File: hardware/eagle/E6_Esp32_TS26C01_v2.brd (EAGLE design)
At the start: 26 x 40 mm, 12 parts, among them J1 ESP32-MEZZAR, J3 ZIF10-5-MOLEX, SW1 KMR221GLFS, U1 ESP32-WROOM-32UE-N16

Commit message: Add files via upload
Other:
- board text added: "1.6"
- board text added: "3.0"
- board text added: "8.0"
